Commit message: [FIX] Resetting with jazzy

File: config/robot_v4.ros2_control.xacro (robot description, xacro)
@@ -50,11 +50,4 @@
                 <state_interface name="velocity"/>
             </joint>
-            <joint name="LJ7">
-                <command_interface name="position"/>
-                <state_interface name="position">
-                  <param name="initial_value">${initial_positions['LJ7']}</param>
-                </state_interface>
-                <state_interface name="velocity"/>
-            </joint>
             <joint name="RJ1">
                 <command_interface name="position"/>
@@ -99,4 +92,11 @@
                 <state_interface name="velocity"/>
             </joint>
+            <joint name="LJ7">
+                <command_interface name="position"/>
+                <state_interface name="position">
+                  <param name="initial_value">${initial_positions['LJ7']}</param>
+                </state_interface>
+                <state_interface name="velocity"/>
+            </joint>
             <joint name="RJ7">
                 <command_interface name="position"/>
